File: PCB/PCB_board_and_schematic/PCB_board_and_schematic.kicad_pcb (KiCad board)
At the start: 2 copper layers, 108.5 x 34.5 mm, 19 parts, among them J1 TangoNano9k_topSide, J2 TangoNano9k_bottomSide, J3 TheSensor, Q1 Q_PMOS_GDS, Q2 Q_PMOS_GDS

Commit message: finished PCB design completly.
Connections:
- J1 pad 3: unconnected-(J1-57-Pad3) -> /Pin_B
- J1 pad 4: unconnected-(J1-56-Pad4) -> /Pin_A
- J1 pad 5: unconnected-(J1-55-Pad5) -> /GMos_A
- J1 pad 6: unconnected-(J1-54-Pad6) -> /GMos_B
Routing:
- net /GMos_B: track 0.00 -> 36.2 mm
- net /GMos_A: track 0.00 -> 32.7 mm
- net /Pin_A: track 0.00 -> 23.2 mm
- net /Pin_B: track 0.00 -> 20.0 mm
Other:
- board text added: "Type-c"
Changed lines of the file:
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@@
 		(capping no)
 		(filling no)
-		(zone_defaults)
 		(pcbplotparams
 			(layerselection 0x00000000_00000000_55555555_5755f5ff)
@@
 			(layers "*.Cu" "*.Mask")
 			(remove_unused_layers no)
-			(net "unconnected-(J1-57-Pad3)")
+			(net "/Pin_B")
 			(pinfunction "57_3")
-			(pintype "passive+no_connect")
+			(pintype "passive")
 		)
 		(pad "4" thru_hole circle
@@
 			(layers "*.Cu" "*.Mask")
 			(remove_unused_layers no)
-			(net "unconnected-(J1-56-Pad4)")
+			(net "/Pin_A")
 			(pinfunction "56_4")
-			(pintype "passive+no_connect")
+			(pintype "passive")
 		)
 		(pad "5" thru_hole circle
@@
 			(layers "*.Cu" "*.Mask")
 			(remove_unused_layers no)
-			(net "unconnected-(J1-55-Pad5)")
+			(net "/GMos_A")
 			(pinfunction "55_5")
-			(pintype "passive+no_connect")
+			(pintype "passive")
 		)
 		(pad "6" thru_hole circle
@@
 			(layers "*.Cu" "*.Mask")
 			(remove_unused_layers no)
-			(net "unconnected-(J1-54-Pad6)")
+			(net "/GMos_B")
 			(pinfunction "54_6")
-			(pintype "passive+no_connect")
+			(pintype "passive")
 		)
 		(pad "7" thru_hole circle
@@
 	)
 	(gr_rect
+		(start 206.5 81.5)
+		(end 209.5 88.5)
+		(stroke
+			(width 0.3)
+			(type dash_dot_dot)
+		)
+		(fill no)
+		(layer "F.SilkS")
+	)
+	(gr_rect
 		(start 137.5 71)
 		(end 150.5 97)
@@
 		)
 	)
+	(gr_text "Type-c"
+		(at 208 85 90)
+		(layer "F.SilkS")
+		(effects
+			(font
+				(size 1 1)
+				(thickness 0.2)
+				(bold yes)
+			)
+		)
+	)
 	(gr_text "Note: You can use a sensor with 3 or 4 pins. \nif it has 3 pins, leave the P_A empty."
 		(at 179.6 100.8 0)
@@
 	)
 	(gr_text "TANG NANO 9K"
-		(at 150 87.7 0)
+		(at 146.298406 87.6 0)
 		(layer "F.SilkS")
 		(effects
@@
 	)
 	(segment
+		(start 121.27 82.124744)
+		(end 121.27 85)
+		(width 0.2)
+		(layer "F.Cu")
+		(net "Net-(D3-A)")
+	)
+	(segment
+		(start 127.94 75.454744)
+		(end 121.27 82.124744)
+		(width 0.2)
+		(layer "F.Cu")
+		(net "Net-(D3-A)")
+	)
+	(segment
+		(start 127.94 72)
+		(end 127.94 75.454744)
+		(width 0.2)
+		(layer "F.Cu")
+		(net "Net-(D3-A)")
+	)
+	(segment
+		(start 112.5 72.25)
+		(end 116.63 72.25)
+		(width 0.2)
+		(layer "F.Cu")
+		(net "Net-(D3-A)")
+	)
+	(segment
+		(start 112.5 74.507057)
+		(end 121.27 83.277057)
+		(width 0.2)
+		(layer "B.Cu")
+		(net "Net-(D3-A)")
+	)
+	(segment
+		(start 121.27 85.46)
+		(end 121.27 85)
+		(width 0.2)
+		(layer "B.Cu")
+		(net "Net-(D3-A)")
+	)
+	(segment
+		(start 112.5 72.25)
+		(end 112.5 74.507057)
+		(width 0.2)
+		(layer "B.Cu")
+		(net "Net-(D3-A)")
+	)
+	(segment
+		(start 121.27 83.277057)
+		(end 121.27 85)
+		(width 0.2)
+		(layer "B.Cu")
+		(net "Net-(D3-A)")
+	)
+	(segment
+		(start 124 88.19)
+		(end 121.27 85.46)
+		(width 0.2)
+		(layer "B.Cu")
+		(net "Net-(D3-A)")
+	)
+	(segment
 		(start 128.71 102.48)
 		(end 128.71 98.55)
@@
 	)
 	(segment
-		(start 123.81 85.63)
-		(end 123.81 85)
+		(start 126.23 92.99)
+		(end 126.23 95.6025)
 		(width 0.2)
 		(layer "F.Cu")
-		(net "Net-(D1-A)")
+		(net "/Mos_A")
 	)
 	(segment
-		(start 127.94 80.87)
-		(end 123.81 85)
+		(start 123.56 100.08)
+		(end 122.08 98.6)
 		(width 0.2)
 		(layer "F.Cu")
-		(net "Net-(D1-A)")
+		(net "/Mos_A")
 	)
 	(segment
-		(start 116.69 77)
-		(end 112.56 77)
+		(start 123.2325 98.6)
+		(end 122.08 98.6)
 		(width 0.2)
 		(layer "F.Cu")
-		(net "Net-(D1-A)")
+		(net "/Mos_A")
 	)
 	(segment
-		(start 121.25 88.19)
-		(end 123.81 85.63)
+		(start 127.17 92.05)
+		(end 126.23 92.99)
 		(width 0.2)
 		(layer "F.Cu")
-		(net "Net-(D1-A)")
+		(net "/Mos_A")
 	)
 	(segment
-		(start 127.94 77)
-		(end 127.94 80.87)
+		(start 123.56 103.75)
+		(end 123.56 100.08)
 		(width 0.2)
 		(layer "F.Cu")
-		(net "Net-(D1-A)")
+		(net "/Mos_A")
 	)
 	(segment
-		(start 123.81 85)
-		(end 123.81 84.12)
+		(start 126.23 95.6025)
+		(end 123.2325 98.6)
 		(width 0.2)
-		(layer "B.Cu")
-		(net "Net-(D1-A)")
+		(layer "F.Cu")
+		(net "/Mos_A")
 	)
 	(segment
-		(start 123.81 84.12)
-		(end 116.69 77)
+		(start 121.25 96.89)
+		(end 119.54 98.6)
 		(width 0.2)
-		(layer "B.Cu")
-		(net "Net-(D1-A)")
+		(layer "F.Cu")
+		(net "Net-(Q1-D)")
 	)
 	(segment
-		(start 121.27 82.124744)
-		(end 121.27 85)
+		(start 121.25 95.81)
+		(end 121.25 96.89)
 		(width 0.2)
 		(layer "F.Cu")
-		(net "Net-(D3-A)")
+		(net "Net-(Q1-D)")
 	)
 	(segment
-		(start 127.94 75.454744)
-		(end 121.27 82.124744)
+		(start 129.79 94.55)
+		(end 127.23 94.55)
 		(width 0.2)
 		(layer "F.Cu")
-		(net "Net-(D3-A)")
+		(net "/Mos_B")
 	)
 	(segment
-		(start 127.94 72)
-		(end 127.94 75.454744)
+		(start 135.06 103.75)
+		(end 135.06 99.82)
 		(width 0.2)
 		(layer "F.Cu")
-		(net "Net-(D3-A)")
+		(net "/Mos_B")
 	)
 	(segment
-		(start 112.5 72.25)
-		(end 116.63 72.25)
+		(start 135.06 99.82)
+		(end 133.79 98.55)
 		(width 0.2)
 		(layer "F.Cu")
-		(net "Net-(D3-A)")
+		(net "/Mos_B")
 	)
 	(segment
-		(start 112.5 74.507057)
-		(end 121.27 83.277057)
+		(start 133.79 98.55)
+		(end 129.79 94.55)
 		(width 0.2)
-		(layer "B.Cu")
-		(net "Net-(D3-A)")
+		(layer "F.Cu")
+		(net "/Mos_B")
 	)
 	(segment
-		(start 121.27 85.46)
-		(end 121.27 85)
+		(start 131.25 98.55)
+		(end 128.51 95.81)
 		(width 0.2)
 		(layer "B.Cu")
-		(net "Net-(D3-A)")
+		(net "Net-(Q2-D)")
 	)
 	(segment
-		(start 112.5 72.25)
-		(end 112.5 74.507057)
+		(start 128.51 95.81)
+		(end 124 95.81)
 		(width 0.2)
 		(layer "B.Cu")
-		(net "Net-(D3-A)")
+		(net "Net-(Q2-D)")
 	)
 	(segment
-		(start 121.27 83.277057)
-		(end 121.27 85)
+		(start 161.99 72.588778)
+		(end 140.028778 94.55)
 		(width 0.2)
-		(layer "B.Cu")
-		(net "Net-(D3-A)")
+		(layer "F.Cu")
+		(net "/GMos_B")
 	)
 	(segment
-		(start 124 88.19)
-		(end 121.27 85.46)
+		(start 140.028778 94.55)
+		(end 134.85 94.55)
 		(width 0.2)
-		(layer "B.Cu")
-		(net "Net-(D3-A)")
+		(layer "F.Cu")
+		(net "/GMos_B")
 	)
 	(segment
-		(start 121.25 96.89)
-		(end 119.54 98.6)
+		(start 123.81 85.63)
+		(end 123.81 85)
 		(width 0.2)
 		(layer "F.Cu")
-		(net "Net-(Q1-D)")
+		(net "Net-(D1-A)")
 	)
 	(segment
-		(start 121.25 95.81)
-		(end 121.25 96.89)
+		(start 127.94 80.87)
+		(end 123.81 85)
 		(width 0.2)
 		(layer "F.Cu")
-		(net "Net-(Q1-D)")
+		(net "Net-(D1-A)")
 	)
 	(segment
-		(start 126.23 92.99)
-		(end 126.23 95.6025)
+		(start 116.69 77)
+		(end 112.56 77)
 		(width 0.2)
 		(layer "F.Cu")
-		(net "/Mos_A")
+		(net "Net-(D1-A)")
 	)
 	(segment
-		(start 123.56 100.08)
-		(end 122.08 98.6)
+		(start 121.25 88.19)
+		(end 123.81 85.63)
 		(width 0.2)
 		(layer "F.Cu")
-		(net "/Mos_A")
+		(net "Net-(D1-A)")
 	)
 	(segment
-		(start 123.2325 98.6)
-		(end 122.08 98.6)
+		(start 127.94 77)
+		(end 127.94 80.87)
 		(width 0.2)
 		(layer "F.Cu")
-		(net "/Mos_A")
+		(net "Net-(D1-A)")
 	)
 	(segment
-		(start 127.17 92.05)
-		(end 126.23 92.99)
+		(start 123.81 85)
+		(end 123.81 84.12)
 		(width 0.2)
-		(layer "F.Cu")
-		(net "/Mos_A")
+		(layer "B.Cu")
+		(net "Net-(D1-A)")
 	)
 	(segment
-		(start 123.56 103.75)
-		(end 123.56 100.08)
+		(start 123.81 84.12)
+		(end 116.69 77)
 		(width 0.2)
-		(layer "F.Cu")
-		(net "/Mos_A")
+		(layer "B.Cu")
+		(net "Net-(D1-A)")
 	)
 	(segment
-		(start 126.23 95.6025)
-		(end 123.2325 98.6)
+		(start 156.91 72.588778)
+		(end 152.498778 77)
 		(width 0.2)
 		(layer "F.Cu")
-		(net "/Mos_A")
+		(net "/Pin_A")
 	)
 	(segment
-		(start 129.79 94.55)
-		(end 127.23 94.55)
+		(start 152.498778 77)
+		(end 135.56 77)
 		(width 0.2)
 		(layer "F.Cu")
-		(net "/Mos_B")
+		(net "/Pin_A")
 	)
 	(segment
-		(start 135.06 103.75)
-		(end 135.06 99.82)
+		(start 139.988778 92.05)
+		(end 134.79 92.05)
 		(width 0.2)
 		(layer "F.Cu")
-		(net "/Mos_B")
+		(net "/GMos_A")
 	)
 	(segment
-		(start 135.06 99.82)
-		(end 133.79 98.55)
+		(start 159.45 72.588778)
+		(end 139.988778 92.05)
 		(width 0.2)
 		(layer "F.Cu")
-		(net "/Mos_B")
+		(net "/GMos_A")
 	)
 	(segment
-		(start 133.79 98.55)
-		(end 129.79 94.55)
+		(start 153.22 73.738778)
+		(end 137.298778 73.738778)
 		(width 0.2)
 		(layer "F.Cu")
-		(net "/Mos_B")
+		(net "/Pin_B")
 	)
 	(segment
-		(start 131.25 98.55)
-		(end 128.51 95.81)
+		(start 137.298778 73.738778)
+		(end 135.56 72)
 		(width 0.2)
-		(layer "B.Cu")
-		(net "Net-(Q2-D)")
+		(layer "F.Cu")
+		(net "/Pin_B")
 	)
 	(segment
-		(start 128.51 95.81)
-		(end 124 95.81)
+		(start 154.37 72.588778)
+		(end 153.22 73.738778)
 		(width 0.2)
-		(layer "B.Cu")
-		(net "Net-(Q2-D)")
+		(layer "F.Cu")
+		(net "/Pin_B")
 	)
 	(zone
